Commit message: Proper SAM prefab

File: Runtime/URDF/sam_auv/sam_auv.urdf (robot description, URDF)
Before this commit: robot sam_auv, 20 links, 19 joints
Links:
- added link rope_link, mass 0.00000001
Joints:
- added joint rope_joint: type fixed, parent base_link, child rope_link, origin xyz=0.540 0.0 0.071 rpy=0.0 0.0 0.0

Commit message: Rope generator works like LinkAttachment now

File: Runtime/URDF/sam_auv/sam_auv.urdf (robot description, URDF)
Before this commit: robot sam_auv, 21 links, 20 joints
Joints:
- joint rope_joint: origin xyz=0.540 0.0 0.071 rpy=0.0 0.0 0.0 -> xyz=0.650 0.0 0.071 rpy=0.0 0.0 0.0
